Commit message: rosa model working

File: models/rosa/omni_wheel.xacro (robot description, xacro)
@@ -1,5 +1,5 @@
 <?xml version="1.0"?>
 <robot xmlns:xacro="http://www.ros.org/wiki/xacro" name="mpo_500">
-  <xacro:macro name="mechanum_wheel" params="name parent *origin">
+  <xacro:macro name="mechanum_wheel" params="name parent dir:='left' *origin">
    <joint name="${name}_joint" type="fixed">
     <insert_block name="origin" />
@@ -20,5 +20,10 @@
      <origin xyz="0 0 0" rpy="0 0 0"/>
      <geometry>
+     <xacro:if value="${dir == 'left'}">
         <mesh filename="package://rosa_description/models/rosa/meshes/MECANUM_WHEEL.dae" scale="0.001 0.001 0.001"/>
+     </xacro:if>
+     <xacro:if value="${dir == 'right'}">
+        <mesh filename="package://rosa_description/models/rosa/meshes/MECANUM_WHEEL.dae" scale="0.001 -0.001 0.001"/>
+     </xacro:if>
      </geometry>
     </visual>
@@ -26,5 +31,5 @@
      <origin xyz="0 0 0" rpy="0 0 0" />
      <geometry>
-        <mesh filename="package://rosa_description/models/rosa/meshes/MECANUM_WHEEL.dae" scale="0.001 0.001 0.001"/>
+        <mesh filename="package://rosa_description/models/rosa/meshes/MECANUM_WHEEL_SIMPLE.stl" scale="0.001 0.001 0.001"/>
      </geometry>
     </collision>

File: models/rosa/rosa.xacro (robot description, xacro)
@@ -9,14 +9,14 @@
   <!-- Wheel Macro -->
   <xacro:mechanum_wheel name="wheel_front_left" parent="base_link">
-  	<origin xyz="0.25 0.28 0.13" rpy="0 0 0" />
+  	<origin xyz="0.34 0.34 0.13" rpy="0 0 0" />
   </xacro:mechanum_wheel>
-  <xacro:mechanum_wheel name="wheel_front_right" parent="base_link">
-  	<origin xyz="0.25 -0.28 0.13" rpy="0 0 3.14" />
+  <xacro:mechanum_wheel name="wheel_front_right" parent="base_link" dir="right">
+  	<origin xyz="0.34 -0.34 0.13" rpy="0 0 0" />
   </xacro:mechanum_wheel>
-  <xacro:mechanum_wheel name="wheel_back_left" parent="base_link">
-  	<origin xyz="-0.25 0.28 0.13" rpy="0 0 0" />
+  <xacro:mechanum_wheel name="wheel_back_left" parent="base_link" dir="right">
+  	<origin xyz="-0.34 0.34 0.13" rpy="0 0 3.14159" />
   </xacro:mechanum_wheel>
   <xacro:mechanum_wheel name="wheel_back_right" parent="base_link">
-  	<origin xyz="-0.25 -0.28 0.13" rpy="0 0 3.14" />
+  	<origin xyz="-0.34 -0.34 0.13" rpy="0 0 3.14159" />
   </xacro:mechanum_wheel>
   <!-- Sensors

File: models/rosa/rosa_body.xacro (robot description, xacro)
@@ -11,5 +11,5 @@
     </inertial>
     <visual>
-      <origin xyz="0. 0. 0" rpy="-1.571 0 1.571" />
+      <origin xyz="0. 0. 0.2" rpy="0 3.14159 0" />
       <geometry>
           <mesh filename="package://rosa_description/models/rosa/meshes/ROSA_BODY.dae" scale="0.001 0.001 0.001"/>
@@ -17,8 +17,8 @@
     </visual>
     <collision>
-      <origin xyz="0. 0. 0.0" rpy="-1.571 0 1.571" />
+      <origin xyz="0. 0. 0.2" rpy="0 3.14159 0" />
       <geometry>
         <!--<box size="0.68 0.41 0.25"/> -->
-         <mesh filename="package://rosa_description/models/rosa/meshes/ROSA_BODY.dae" scale="0.001 0.001 0.001"/>
+         <mesh filename="package://rosa_description/models/rosa/meshes/ROSA_BODY_SIMPLE.stl" scale="0.001 0.001 0.001"/>
       </geometry>
     </collision>

Commit message: fixing scales and orientation

File: models/rosa/omni_wheel.xacro (robot description, xacro)
@@ -3,5 +3,5 @@
   <xacro:macro name="mechanum_wheel" params="name parent dir:='left' *origin">
    <joint name="${name}_joint" type="fixed">
-    <insert_block name="origin" />
+    <xacro:insert_block name="origin" />
     <axis xyz="0 1 0" />
     <joint_properties damping="1" friction="1" />

File: models/rosa/rosa_body.xacro (robot description, xacro)
@@ -4,6 +4,6 @@
   <link name="${name}">
     <inertial>
-      <mass value="200"/>
-      <origin xyz="0 0 0" />
+      <mass value="400"/>
+      <origin xyz="0 0 0.5" />
        <inertia ixx="5.652232699207" ixy="0.009719934438" ixz="1.293988226423"
                iyy="5.669473158652" iyz="0.007379583694"
@@ -11,14 +11,14 @@
     </inertial>
     <visual>
-      <origin xyz="0. 0. 0.2" rpy="0 3.14159 0" />
+      <origin xyz="0. 0. 0.2" rpy="0 3.14159 3.14159" />
       <geometry>
-          <mesh filename="package://rosa_description/models/rosa/meshes/ROSA_BODY.dae" scale="0.001 0.001 0.001"/>
+          <mesh filename="package://rosa_description/models/rosa/meshes/ROSA_BODY.dae" scale="1.0 1.0 1.0"/>
       </geometry>
     </visual>
     <collision>
-      <origin xyz="0. 0. 0.2" rpy="0 3.14159 0" />
+      <origin xyz="0. 0. 0.2" rpy="0 3.14159 3.14159" />
       <geometry>
         <!--<box size="0.68 0.41 0.25"/> -->
-         <mesh filename="package://rosa_description/models/rosa/meshes/ROSA_BODY_SIMPLE.stl" scale="0.001 0.001 0.001"/>
+         <mesh filename="package://rosa_description/models/rosa/meshes/ROSA_BODY_SIMPLE.stl" scale="1.0 1.0 1.0"/>
       </geometry>
     </collision>

Commit message: update

File: models/rosa/omni_wheel.xacro (robot description, xacro)
@@ -1,6 +1,35 @@
 <?xml version="1.0"?>
 <robot xmlns:xacro="http://www.ros.org/wiki/xacro" name="rosa">
-  <xacro:macro name="mechanum_wheel" params="name parent dir:='left' *origin">
-   <joint name="${name}_joint" type="fixed">
+  <xacro:macro name="mechanum_wheel" params="name parent reflect:='false' *origin">
+   <link name="${name}_link" type="wheel">
+    <inertial>
+      <mass value="1.0" />
+      <origin xyz="0 0 0" rpy="0 0 0" />
+        <inertia  ixx="0.04" ixy="0.0007" ixz="0.0"
+                  iyy="0.02" iyz="0.004"
+                  izz="0.05" />
+    </inertial>
+    <visual>
+     <geometry>
+     <xacro:if value="${reflect}">
+        <mesh filename="package://rosa_description/models/rosa/meshes/MECANUM_WHEEL.dae" scale="0.001 -0.001 0.001"/>
+     </xacro:if>
+     <xacro:unless value="${reflect}">
+        <mesh filename="package://rosa_description/models/rosa/meshes/MECANUM_WHEEL.dae" scale="0.001 0.001 0.001"/>
+     </xacro:unless>
+     </geometry>
+    </visual>
+    <collision>
+     <!-- if using mess instead cylinder, xyz = 0 rpy=0 -->
+     <origin xyz="0 0 0" rpy="1.5707 0 0"/>
+     <geometry>
+        <!--
+        <mesh filename="package://rosa_description/models/rosa/meshes/MECANUM_WHEEL_SIMPLE.stl" scale="0.001 0.001 0.001"/>
+        -->
+	<cylinder length="0.12" radius="0.12"/>
+     </geometry>
+    </collision>
+   </link>
+   <joint name="${name}_joint" type="continuous">
     <xacro:insert_block name="origin" />
     <axis xyz="0 1 0" />
@@ -9,35 +38,7 @@
     <child link="${name}_link" />
    </joint>
-   <link name="${name}_link" type="wheel">
-    <inertial>
-      <mass value="8.9" />
-      <origin xyz="0 0 0" rpy="0 0 0" />
-        <inertia  ixx="0.04" ixy="0.0007" ixz="0.0"
-                  iyy="0.02" iyz="0.004"
-                  izz="0.05" />
-    </inertial>
-    <visual>
-     <origin xyz="0 0 0" rpy="0 0 0"/>
-     <geometry>
-     <xacro:if value="${dir == 'left'}">
-        <mesh filename="package://rosa_description/models/rosa/meshes/MECANUM_WHEEL.dae" scale="0.001 0.001 0.001"/>
-     </xacro:if>
-     <xacro:if value="${dir == 'right'}">
-        <mesh filename="package://rosa_description/models/rosa/meshes/MECANUM_WHEEL.dae" scale="0.001 -0.001 0.001"/>
-     </xacro:if>
-     </geometry>
-    </visual>
-    <collision>
-     <origin xyz="0 0 0" rpy="0 0 0" />
-     <geometry>
-        <mesh filename="package://rosa_description/models/rosa/meshes/MECANUM_WHEEL_SIMPLE.stl" scale="0.001 0.001 0.001"/>
-     </geometry>
-    </collision>
-   </link>
   <gazebo reference="${name}_link">
-    <mu1 value="2.6"/>
-    <mu2 value="2.6"/>
-    <kp value="100000.0" />
-    <kd value="10.0" />
+    <mu1 value="1"/>
+    <mu2 value="1"/>
   </gazebo>
   </xacro:macro>

File: models/rosa/rosa.xacro (robot description, xacro)
@@ -1,7 +1,11 @@
 <?xml version="1.0" ?>
 <robot name="rosa" xmlns:xacro="http://www.ros.org/wiki/xacro">
+  <xacro:include filename="materials.xacro" />
   <xacro:include filename="rosa_gazebo.xacro" />
   <xacro:include filename="omni_wheel.xacro" />
   <xacro:include filename="rosa_body.xacro" />
+<xacro:property name="wheel_x" value="0.34" />
+<xacro:property name="wheel_y" value="0.34" />
+<xacro:property name="wheel_z" value="0.13" />
   <!-- Base Macro-->
   <xacro:rosa_base name="base_link">
@@ -9,19 +13,21 @@
   <!-- Wheel Macro -->
   <xacro:mechanum_wheel name="wheel_front_left" parent="base_link">
-  	<origin xyz="0.34 0.34 0.13" rpy="0 0 0" />
+  	<origin xyz="${wheel_x} ${wheel_y} ${wheel_z}" rpy="0 0 0" />
   </xacro:mechanum_wheel>
-  <xacro:mechanum_wheel name="wheel_front_right" parent="base_link" dir="right">
-  	<origin xyz="0.34 -0.34 0.13" rpy="0 0 0" />
+  <xacro:mechanum_wheel name="wheel_front_right" parent="base_link" reflect="true">
+  	<origin xyz="${wheel_x} -${wheel_y} ${wheel_z}" rpy="0 0 0" />
   </xacro:mechanum_wheel>
-  <xacro:mechanum_wheel name="wheel_back_left" parent="base_link" dir="right">
-  	<origin xyz="-0.34 0.34 0.13" rpy="0 0 3.14159" />
+  <xacro:mechanum_wheel name="wheel_back_left" parent="base_link" reflect="true">
+  	<origin xyz="-${wheel_x} ${wheel_y} ${wheel_z}" rpy="0 0 3.14159" />
   </xacro:mechanum_wheel>
   <xacro:mechanum_wheel name="wheel_back_right" parent="base_link">
-  	<origin xyz="-0.34 -0.34 0.13" rpy="0 0 3.14159" />
+  	<origin xyz="-${wheel_x} -${wheel_y} ${wheel_z}" rpy="0 0 3.14159" />
   </xacro:mechanum_wheel>
-  <!-- Sensors
-  <xacro:sick_laser_v0 name="lidar_1" parent="base_link" ros_topic="lidar_1/scan_filtered">
-    <origin xyz="0.442 0 0.372" rpy="0 0 0" />
-  </xacro:sick_laser_v0>
--->
+<!-- Robot Footprint -->
+  <link name="base_footprint"/>
+  <joint name="base_joint" type="fixed">
+    <parent link="base_link"/>
+    <child link="base_footprint"/>
+    <origin xyz="0.0 0.0 -${wheel_z}" rpy="0 0 0"/>
+  </joint>
 </robot>

File: models/rosa/rosa_body.xacro (robot description, xacro)
@@ -4,6 +4,6 @@
   <link name="${name}">
     <inertial>
-      <mass value="400"/>
-      <origin xyz="0 0 0.5" />
+      <mass value="80"/>
+      <origin xyz="0 0 0.3" />
        <inertia ixx="5.652232699207" ixy="0.009719934438" ixz="1.293988226423"
                iyy="5.669473158652" iyz="0.007379583694"
@@ -13,12 +13,12 @@
       <origin xyz="0. 0. 0.2" rpy="0 3.14159 3.14159" />
       <geometry>
-          <mesh filename="package://rosa_description/models/rosa/meshes/ROSA_BODY.dae" scale="1.0 1.0 1.0"/>
+          <mesh filename="package://rosa_description/models/rosa/meshes/ROSA_BODY.dae"/>
       </geometry>
+      <material name="white"/>
     </visual>
     <collision>
       <origin xyz="0. 0. 0.2" rpy="0 3.14159 3.14159" />
       <geometry>
-        <!--<box size="0.68 0.41 0.25"/> -->
-         <mesh filename="package://rosa_description/models/rosa/meshes/ROSA_BODY_SIMPLE.stl" scale="1.0 1.0 1.0"/>
+         <mesh filename="package://rosa_description/models/rosa/meshes/ROSA_BODY_SIMPLE.stl"/>
       </geometry>
     </collision>

File: models/rosa/rosa_gazebo.xacro (robot description, xacro)
@@ -21,47 +21,3 @@
     <self_collide>false</self_collide>
   </gazebo>
-  <gazebo reference="lidar_1_link">
-      <sensor type="ray" name="lidar_1_sensor">
-          <pose>0 0 0 0 0 0</pose>
-          <visualize>false</visualize>
-          <update_rate>40</update_rate>
-          <ray>
-            <scan>
-              <horizontal>
-                <samples>720</samples>
-                <resolution>1</resolution>
-                <min_angle>-1.48353</min_angle>
-                <max_angle>1.48353</max_angle>
-              </horizontal>
-            </scan>
-            <range>
-              <min>0.10</min>
-              <max>30.0</max>
-              <resolution>0.05</resolution>
-            </range>
-            <noise>
-              <type>gaussian</type>
-              <!-- Noise parameters based on published spec for Hokuyo laser
-                   achieving "+-30mm" accuracy at range < 10m.  A mean of 0.0m and
-                   stddev of 0.01m will put 99.7% of samples within 0.03m of the true
-                   reading. -->
-              <mean>0.0</mean>
-              <stddev>0.01</stddev>
-            </noise>
-          </ray>
-          <plugin name="lidar_1" filename="libgazebo_ros_laser.so">
-            <topicName>lidar_1/scan_filtered</topicName>
-            <frameName>lidar_1_link</frameName>
-          </plugin>
-        </sensor>
-  </gazebo>
-  <gazebo>
-    <plugin name="rosa_controller" filename="libgazebo_ros_planar_move.so">
-      <commandTopic>cmd_vel</commandTopic>
-      <odometryTopic>odom</odometryTopic>
-      <odometryFrame>odom</odometryFrame>
-      <odometryRate>20.0</odometryRate>
-      <robotBaseFrame>base_link</robotBaseFrame>
-    </plugin>
-  </gazebo>
 </robot>

Commit message: rviz & gz working properly

File: models/rosa/omni_wheel.xacro (robot description, xacro)
@@ -13,23 +13,19 @@
      <geometry>
      <xacro:if value="${reflect}">
-        <mesh filename="package://rosa_description/models/rosa/meshes/MECANUM_WHEEL.dae" scale="0.001 -0.001 0.001"/>
+        <mesh filename="file://$(find rosa_description)/models/rosa/meshes/MECANUM_WHEEL_mhg.dae" scale="1 -1 1"/>
      </xacro:if>
      <xacro:unless value="${reflect}">
-        <mesh filename="package://rosa_description/models/rosa/meshes/MECANUM_WHEEL.dae" scale="0.001 0.001 0.001"/>
+        <mesh filename="file://$(find rosa_description)/models/rosa/meshes/MECANUM_WHEEL_mhg.dae" scale="1 1 1"/>
      </xacro:unless>
      </geometry>
     </visual>
     <collision>
-     <!-- if using mess instead cylinder, xyz = 0 rpy=0 -->
      <origin xyz="0 0 0" rpy="1.5707 0 0"/>
      <geometry>
-        <!--
-        <mesh filename="package://rosa_description/models/rosa/meshes/MECANUM_WHEEL_SIMPLE.stl" scale="0.001 0.001 0.001"/>
-        -->
-	<cylinder length="0.12" radius="0.12"/>
+	<cylinder length="0.06" radius="0.075"/>
      </geometry>
     </collision>
    </link>
-   <joint name="${name}_joint" type="continuous">
+   <joint name="${name}_joint" type="fixed">
     <xacro:insert_block name="origin" />
     <axis xyz="0 1 0" />

File: models/rosa/rosa.xacro (robot description, xacro)
@@ -5,7 +5,7 @@
   <xacro:include filename="omni_wheel.xacro" />
   <xacro:include filename="rosa_body.xacro" />
-<xacro:property name="wheel_x" value="0.34" />
-<xacro:property name="wheel_y" value="0.34" />
-<xacro:property name="wheel_z" value="0.13" />
+<xacro:property name="wheel_x" value="0.35" />
+<xacro:property name="wheel_y" value="0.295" />
+<xacro:property name="wheel_z" value="0.075" />
   <!-- Base Macro-->
   <xacro:rosa_base name="base_link">

File: models/rosa/rosa_body.xacro (robot description, xacro)
@@ -11,14 +11,14 @@
     </inertial>
     <visual>
-      <origin xyz="0. 0. 0.2" rpy="0 3.14159 3.14159" />
+      <origin xyz="0. 0. 0.15" rpy="0 3.14159 3.14159" />
       <geometry>
-          <mesh filename="package://rosa_description/models/rosa/meshes/ROSA_BODY.dae"/>
+          <mesh filename="file://$(find rosa_description)/models/rosa/meshes/ROSA_BODY.dae"/>
       </geometry>
       <material name="white"/>
     </visual>
     <collision>
-      <origin xyz="0. 0. 0.2" rpy="0 3.14159 3.14159" />
+      <origin xyz="0. 0. 0.15" rpy="0 3.14159 3.14159" />
       <geometry>
-         <mesh filename="package://rosa_description/models/rosa/meshes/ROSA_BODY_SIMPLE.stl"/>
+         <mesh filename="file://$(find rosa_description)/models/rosa/meshes/ROSA_BODY_SIMPLE.stl"/>
       </geometry>
     </collision>
