Commit message: great updates

File: description/rosa/omni_wheel.xacro (robot description, xacro)
@@ -4,5 +4,5 @@
    <link name="${name}_link" type="wheel">
     <inertial>
-      <mass value="1.0" />
+      <mass value="0.25" />
       <origin xyz="0 0 0" rpy="0 0 0" />
         <inertia  ixx="0.04" ixy="0.0007" ixz="0.0"
@@ -30,11 +30,11 @@
     <xacro:insert_block name="origin" />
     <axis xyz="0 1 0" />
-    <joint_properties damping="1" friction="1" />
+    <joint_properties damping="0.01" friction="0.01" />
     <parent link="${parent}" />
     <child link="${name}_link" />
    </joint>
   <gazebo reference="${name}_link">
-    <mu1 value="1"/>
-    <mu2 value="1"/>
+    <mu1 value="0.1"/>
+    <mu2 value="0.1"/>
   </gazebo>
   </xacro:macro>

File: description/rosa/rosa.xacro (robot description, xacro)
@@ -5,4 +5,5 @@
   <xacro:include filename="omni_wheel.xacro" />
   <xacro:include filename="rosa_body.xacro" />
+  <xacro:include filename="realsense_d435.xacro" />
 <xacro:property name="wheel_x" value="0.35" />
 <xacro:property name="wheel_y" value="0.295" />
@@ -24,11 +25,18 @@
   	<origin xyz="-${wheel_x} -${wheel_y} 0" rpy="0 0 3.14159" />
   </xacro:mechanum_wheel>
+ <!-- ========= -->
+    <!-- 3D CAMERA -->
+    <!-- =========
+    <xacro:realsense_d435 name="realsense_head" parent="base_link">
+        <origin xyz="0.425 0.0 1.59" rpy="0.0 0.0 0.0"/>
+    </xacro:realsense_d435>
+    -->
 <!-- Robot Footprint -->
   <link name="base_footprint"/>
   <link name="base_link"/>
   <joint name="footprint_joint" type="fixed">
-    <parent link="base_link"/>
-    <child link="base_footprint"/>
-    <origin xyz="0.0 0.0 -${wheel_z}" rpy="0 0 0"/>
+    <parent link="base_footprint"/>
+    <child link="base_link"/>
+    <origin xyz="0.0 0.0 ${wheel_z}" rpy="0 0 0"/>
   </joint>
   <joint name="chasis_joint" type="fixed">

File: description/rosa/rosa_gazebo.xacro (robot description, xacro)
@@ -21,3 +21,22 @@
     <self_collide>false</self_collide>
   </gazebo>
+<gazebo>
+    <plugin name="rosa_controller" filename="libgazebo_ros_omni_drive.so">
+      <commandTopic>cmd_vel</commandTopic>
+      <odometryTopic>odom</odometryTopic>
+      <odometryFrame>odom</odometryFrame>
+      <odometryRate>20.0</odometryRate>
+      <robotBaseFrame>base_footprint</robotBaseFrame>
+      <wheel_radius>0.075</wheel_radius>
+      <base_length>0.65</base_length>
+      <base_width>0.65</base_width>
+      <front_left_joint>wheel_front_left_joint</front_left_joint>
+      <front_right__joint>wheel_front_right_joint</front_right__joint>
+      <rear_left_joint>wheel_back_left_joint</rear_left_joint>
+      <rear_right_joint>wheel_back_right_joint</rear_right_joint>
+      <wheel_max_speed> 20.0 </wheel_max_speed>
+      <wheel_acceleration> 10.0</wheel_acceleration>
+      <joint_config>1 1 -1 -1</joint_config>
+    </plugin>
+  </gazebo>
 </robot>
