Commit message: Added LiDAR sensor to the gazebo model and slam_launch.py to start SLAM mapping, also added a rviz config to set the program for the mapping

File: description/rosa/rosa.xacro (robot description, xacro)
@@ -6,4 +6,5 @@
   <xacro:include filename="rosa_body.xacro" />
   <xacro:include filename="realsense_d435.xacro" />
+  <xacro:include filename="lidar_sensor.xacro"/>
 <xacro:property name="wheel_x" value="0.35" />
 <xacro:property name="wheel_y" value="0.295" />
@@ -32,4 +33,8 @@
     </xacro:realsense_d435>
     -->
+  <!-- Sensor LiDAR -->
+  <xacro:lidar_sensor name="lidar_sensor" parent="base_link">
+    <origin xyz="0.53 0.0 0.01" rpy="0 0 0"/>
+  </xacro:lidar_sensor>
 <!-- Robot Footprint -->
   <link name="base_footprint"/>
