Commit message: -Added depth camera frames acording to hardware -Modified laser and slam params -Added .yaml for navigation params -Created amcl launcher for navigation and slam

File: description/rosa/lidar_sensor.xacro (robot description, xacro)
@@ -28,5 +28,5 @@
       <sensor type="ray" name="${name}">
       <visualize>true</visualize>
-        <update_rate>40</update_rate>
+        <update_rate>20</update_rate>
         <ray>
           <scan>
@@ -34,10 +34,10 @@
               <samples>1440</samples>
               <resolution>0.25*(360/1440)</resolution>
-              <min_angle>-2.5307</min_angle>
-              <max_angle>2.5307</max_angle>
+              <min_angle>-1.5307</min_angle>
+              <max_angle>1.5307</max_angle>
             </horizontal>
           </scan>
           <range>
-            <min>0.7</min>
+            <min>0.07</min>
             <max>30.0</max>
             <resolution>0.1</resolution>

File: description/rosa/realsense_d435.xacro (robot description, xacro)
@@ -32,7 +32,7 @@
             <xacro:insert_block name="origin" />
             <parent link="${parent}"/>
-            <child link="${name}_d435_link" />
+            <child link="${name}_link" />
         </joint>
-        <link name="${name}_d435_link">
+        <link name="${name}_link">
             <visual>
                 <origin xyz="${d435_cam_mount_from_center_offset} 0.0 ${d435_cam_height/2}" rpy="${pi/2} 0 ${pi/2}"/>
@@ -56,20 +56,34 @@
         </link>
         <!-- camera depth joints and links -->
-        <joint name="${name}_depth_camera_joint" type="fixed">
+        <joint name="${name}_depth_joint" type="fixed">
             <origin xyz="${d435_cam_depth_px} ${d435_cam_depth_py} ${d435_cam_depth_pz}" rpy="0 0 0"/>
-            <parent link="${name}_d435_link"/>
-            <child link="${name}_depth_camera_frame" />
+            <parent link="${name}_link"/>
+            <child link="${name}_depth_frame" />
         </joint>
-        <link name="${name}_depth_camera_frame"/>
-        <joint name="${name}_camera_optical_joint" type="fixed">
+        <link name="${name}_depth_frame"/>
+        <joint name="${name}_depth_optical_joint" type="fixed">
             <origin xyz="0.02 0 0" rpy="${-pi/2} 0 ${-pi/2}" />
-            <parent link="${name}_depth_camera_frame" />
-            <child link="${name}_camera_optical_frame" />
+            <parent link="${name}_depth_frame" />
+            <child link="${name}_depth_optical_frame" />
         </joint>
-        <link name="${name}_camera_optical_frame"/>
-        <gazebo reference="${name}_d435_link">
-            <sensor type="depth" name="${name}_depth_sensor">
+        <link name="${name}_depth_optical_frame"/>
+        <!-- camera color joints and links -->
+        <joint name="${name}_color_joint" type="fixed">
+            <origin xyz="${d435_cam_depth_px} ${d435_cam_depth_py} ${d435_cam_depth_pz}" rpy="0 0 0"/>
+            <parent link="${name}_link"/>
+            <child link="${name}_color_frame" />
+        </joint>
+        <link name="${name}_color_frame"/>
+        <joint name="${name}_color_optical_joint" type="fixed">
+            <origin xyz="0.02 0 0" rpy="${-pi/2} 0 ${-pi/2}" />
+            <parent link="${name}_color_frame" />
+            <child link="${name}_color_optical_frame" />
+        </joint>
+        <link name="${name}_color_optical_frame"/>
+        <gazebo reference="${name}_link">
+            <sensor type="depth" name="${name}">
+                <visualize>true</visualize>
                 <update_rate>10.0</update_rate>
-                <camera name="${name}_camera">
+                <camera name="${name}_depth_camera">
                     <horizontal_fov>1.21</horizontal_fov>
                     <image>
@@ -87,5 +101,5 @@
                     <alwaysOn>true</alwaysOn>
                     <updateRate>0.0</updateRate>
-                    <frame_name>${name}_camera_optical_frame</frame_name>
+                    <frame_name>${name}_depth_optical_frame</frame_name>
                     <pointCloudCutoff>0.105</pointCloudCutoff>
                     <pointCloudCutoffMax>10.0</pointCloudCutoffMax>
@@ -101,9 +115,9 @@
                     <hackBaseline>0</hackBaseline>
                     <ros>
-        		<imageTopicName>${name}/image_raw</imageTopicName>
-        		<cameraInfoTopicName>${name}/camera_info</cameraInfoTopicName>
-        		<depthImageTopicName>${name}/depth_image_raw</depthImageTopicName>
-        		<pointCloudTopicName>${name}/points</pointCloudTopicName>
-     		    </ros>
+                        <imageTopicName>${name}/image_raw</imageTopicName>
+                        <cameraInfoTopicName>${name}/camera_info</cameraInfoTopicName>
+                        <depthImageTopicName>${name}/depth_image_raw</depthImageTopicName>
+                        <pointCloudTopicName>${name}/points</pointCloudTopicName>
+     		        </ros>
                 </plugin>
             </sensor>

File: description/rosa/rosa.xacro (robot description, xacro)
@@ -28,5 +28,5 @@
  <!-- ========= -->
     <!-- 3D CAMERA -->
-    <xacro:realsense_d435 name="realsense_head" parent="base_link">
+    <xacro:realsense_d435 name="camera" parent="base_link">
         <origin xyz="0.425 0.0 1.59" rpy="0.0 0.0 0.0"/>
     </xacro:realsense_d435>
